File: pcb/thumb-unit-left/thumb-unit-left.kicad_sch (KiCad schematic)
At the start: 24 parts, among them J1 Conn_01x10, SW1 SW_SPDT, SW2 SW_Push, SW3 SW_Push, SW4 SW_Push, SW5 SW_Push, U1 xiao-ble, U2 PMW3610, U3 TLV70218_SOT23-5

Commit message: fix(pcb/thumb-unit-left): GND pour, swap to roBa XIAO footprint, clean routing
- Schematic: switch U1 footprint to mcu_roba:XIAO_nRF52840_wBAT_wNFC_1
  to match the right half (same schematic file structure; the two
  halves only differ in PCB).
- PCB: add B.Cu GND zone (SMD side for the left half is the bottom
  layer) and remove F.Cu↔B.Cu stitching vias that were blocking the
  zone from reaching C2 / J1 / U3 GND pads.
- PCB: route +3V3, +1V8, the SPI bus (SDIO/SCLK/MOTION/NCS), the
  keyboard matrix (ROW0-3 × COL0-4), the trackball charge-pump and
  VCSEL nets, and the BAT_SW power switch path so all nets resolve.

DRC: 0 unconnected, 0 schematic-parity errors. Remaining warnings are
identical in kind to the right half (environment-only and intentional
edge clearances on U1 pads 19-22).

Co-Authored-By: Claude Opus 4.7 (1M context) <noreply@anthropic.com>
Parts:
- U1: footprint mcu:xiao-ble-tht -> mcu_roba:XIAO_nRF52840_wBAT_wNFC_1
Connections:
- net GND: no longer U1.18 (GND)
- no-connect marks 5 -> 6
Changed lines of the file:
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@@
+	)
+	(no_connect
+		(at 85.09 60.96)
 	)
 	(no_connect
@@
 			)
 		)
-		(property "Footprint" "mcu:xiao-ble-tht"
+		(property "Footprint" "mcu_roba:XIAO_nRF52840_wBAT_wNFC_1"
 			(at 73.66 71.12 0)
 			(effects
@@
 					(unit 1)
 				)
-			)
-		)
-	)
-	(symbol
-		(lib_id "power:GND")
-		(at 85.09 60.96 180)
-		(unit 1)
-		(exclude_from_sim no)
-		(in_bom yes)
-		(on_board yes)
-		(dnp no)
-		(fields_autoplaced yes)
-		(property "Reference" "#PWR05"
-			(at 85.09 54.61 0)
-			(effects
-				(font
-					(size 1.27 1.27)
-				)
-				(hide yes)
-			)
-		)
-		(property "Value" "GND"
-			(at 85.09 55.88 0)
-			(effects
-				(font
-					(size 1.27 1.27)
-				)
-			)
-		)
-		(property "Footprint" ""
-			(at 85.09 60.96 0)
-			(effects
-				(font
-					(size 1.27 1.27)
-				)
-				(hide yes)
-			)
-		)
-		(property "Datasheet" ""
-			(at 85.09 60.96 0)
-			(effects
-				(font
-					(size 1.27 1.27)
-				)
-				(hide yes)
-			)
-		)
-		(property "Description" "Power symbol creates a global label with name \"GND\" , ground"
-			(at 85.09 60.96 0)
-			(effects
-				(font
-					(size 1.27 1.27)
-				)
-				(hide yes)
-			)
-		)
-		(pin "1"
-		)
-		(instances
-			(project ""
-				(path "/8578c350-a4e6-49ba-a463-553b48512071"
-					(reference "#PWR05")
-					(unit 1)
-				)
